Commit message: update joint limits to current measured joint limits

File: config/urdf/hdt.xacro (robot description, xacro)
@@ -21,5 +21,6 @@
             <parent link="${mounting_link}"/>
             <child link="arm_1_shoulder_twist_link"/>
-            <limit lower="${-175*degrees}" upper="${175*degrees}" effort="10" velocity="0.38"/>
+            <!-- <limit lower="${-175*degrees}" upper="${175*degrees}" effort="10" velocity="0.38"/>  -->
+            <limit lower="${-120*degrees}" upper="${120*degrees}" effort="10" velocity="0.38"/>
             <axis xyz="0 0 1"/>
             <origin xyz="${mounting_origin}"/>
@@ -51,7 +52,6 @@
             <parent link="arm_1_shoulder_twist_link"/>
             <child link="arm_2_shoulder_lift_link"/>
-            <limit lower="${-125*degrees}" upper="${125*degrees}" effort="10" velocity="0.38"/>
-            <!-- safety controller not working... makes the arm very weak!! -->
-            <!-- <safety_controller k_position="2000" k_velocity="1.5" soft_lower_limit="${-125*degrees}" soft_upper_limit="${125*degrees}"/> -->
+            <!-- <limit lower="${-125*degrees}" upper="${125*degrees}" effort="10" velocity="0.38"/> -->
+            <limit lower="${-110*degrees}" upper="${110*degrees}" effort="10" velocity="0.38"/>
             <axis xyz="0 0 -1"/>
             <origin xyz="0.0 0.0 ${length1}" rpy="${pi/2} 0 0"/>
@@ -83,5 +83,6 @@
             <parent link="arm_2_shoulder_lift_link"/>
             <child link="arm_3_elbow_twist_link"/>
-            <limit lower="${-175*degrees}" upper="${175*degrees}" effort="10" velocity="0.38"/>
+            <!-- <limit lower="${-175*degrees}" upper="${175*degrees}" effort="10" velocity="0.38"/> -->
+            <limit lower="${-150*degrees}" upper="${150*degrees}" effort="10" velocity="0.38"/>
             <axis xyz="0 0 1" />
             <origin xyz="0.0 0.0 0.0" rpy="${-pi/2} 0 0" />
@@ -113,7 +114,7 @@
             <parent link="arm_3_elbow_twist_link"/>
             <child link="arm_4_elbow_lift_link"/>
-            <limit lower="${-125*degrees}" upper="${125*degrees}" effort="10" velocity="0.38"/>
+            <!-- <limit lower="${-125*degrees}" upper="${125*degrees}" effort="10" velocity="0.38"/> -->
+            <limit lower="${-110*degrees}" upper="${110*degrees}" effort="10" velocity="0.38"/>
             <axis xyz="0 0 -1"/>
-            <!-- <origin xyz="0.0 0.0 ${length3}" rpy="${pi/2} ${pi/2} 0"/> -->
             <origin xyz="0.0 0.0 ${length3}" rpy="${pi/2} ${pi/2} 0"/>
             <dynamics damping="10" friction="0.1"/>
@@ -142,5 +143,6 @@
             <parent link="arm_4_elbow_lift_link"/>
             <child link="arm_5_wrist_twist_link"/>
-            <limit lower="${-90*degrees}" upper="${90*degrees}" effort="10" velocity="0.38"/>
+            <!-- <limit lower="${-90*degrees}" upper="${90*degrees}" effort="10" velocity="0.38"/> -->
+            <limit lower="${-85*degrees}" upper="${85*degrees}" effort="10" velocity="0.38"/>
             <axis xyz="0 0 1"/>
             <origin xyz="0.0 0.0 ${length4}" rpy="${-pi/2} 0 0"/>
@@ -172,6 +174,6 @@
             <parent link="arm_5_wrist_twist_link"/>
             <child link="arm_6_wrist_lift_link"/>
-            <limit lower="${-60*degrees}" upper="${60*degrees}" effort="10" velocity="0.38"/>
-            <!--   <safety_controller k_position="100" k_velocity="1.5" soft_lower_limit="${-59*degrees}" soft_upper_limit="${59*degrees}"/> -->
+            <!-- <limit lower="${-60*degrees}" upper="${60*degrees}" effort="10" velocity="0.38"/> -->
+            <limit lower="${-40*degrees}" upper="${40*degrees}" effort="10" velocity="0.38"/>
             <axis xyz="0 0 -1"/>
             <origin xyz="0.0 0.0 ${length5}" rpy="${pi/2} -${pi/2} 0"/>
@@ -202,5 +204,6 @@
             <parent link="arm_6_wrist_lift_link"/>
             <child link="arm_7_gripper_lift_link"/>
-            <limit lower="${-60*degrees}" upper="${60*degrees}" effort="10" velocity="0.38"/>
+            <!-- <limit lower="${-60*degrees}" upper="${60*degrees}" effort="10" velocity="0.38"/> -->
+            <limit lower="${-55*degrees}" upper="${55*degrees}" effort="10" velocity="0.38"/>
             <axis xyz="0 0 1"/>
             <origin xyz="${length6} 0 0" rpy="${-pi/2} 0 0"/>
