Commit message: correct finger joint frames and joint axes

File: config/urdf/fake_gripper.xacro (robot description, xacro)
@@ -43,5 +43,6 @@
             <limit lower="0.001" upper="0.042" effort="45" velocity="0.38"/>
             <axis xyz="0 0 1"/>
-            <origin xyz="${0.5 * (gripper_base_length + finger_length)} 0 ${0.5 * (gripper_base_height - finger_height)}"/>
+            <origin xyz="${0.5 * (gripper_base_length + finger_length)} 0 ${-0.5 * (gripper_base_height - finger_height)}"
+                    rpy="0 0 0"/>
             <dynamics damping="10" friction="0.1"/>
         </joint>
@@ -67,6 +68,7 @@
             <child link="finger_link2"/>
             <limit lower="0.001" upper="0.042" effort="45" velocity="0.38"/>
-            <axis xyz="0 0 -1"/>
-            <origin xyz="${0.5 * (gripper_base_length + finger_length)} 0 ${-0.5 * (gripper_base_height - finger_height)}"/>
+            <axis xyz="0 0 1"/>
+            <origin xyz="${0.5 * (gripper_base_length + finger_length)} 0 ${0.5 * (gripper_base_height - finger_height)}"
+                    rpy="${pi} 0 0"/>
             <dynamics damping="10" friction="0.1"/>
         </joint>
