Commit message: v3 of measured hdt model parameters

File: config/urdf/andalite.xacro (robot description, xacro)
@@ -7,8 +7,16 @@
     <include filename="$(find hdt)/config/urdf/shelf.xacro"/>
     <include filename="$(find hdt)/config/urdf/kinect.xacro"/>
-    <xacro:property name="shelf_dist_from_bumper_m" value="0.10795" />
-    <xacro:property name="bumper_to_rail_bottom_offset_z" value="0.132" />
-    <!-- <xacro:property name="rail_width" value="0.421" />  -->    <!-- values computed from diagrams -->
-    <xacro:property name="rail_width" value="0.418" />              <!-- values measured from husky at lab -->
+    <!-- values computed from diagrams -->
+    <!-- <xacro:property name="rail_width" value="0.421" />  -->
+    <!-- <xacro:property name="shelf_dist_from_bumper_m" value="0.10795" /> -->
+    <!-- <xacro:property name="bumper_to_rail_bottom_offset_z" value="0.132" /> -->
+    <!-- values measured from husky at lab -->
+    <!-- <xacro:property name="rail_width" value="0.418" /> -->
+    <!-- <xacro:property name="shelf_dist_from_bumper_m" value="0.10795" /> -->
+    <!-- <xacro:property name="bumper_to_rail_bottom_offset_z" value="0.132" /> -->
+    <!-- values measured on 2014-07-08 (and averaged with previous values) -->
+    <xacro:property name="rail_width" value="0.419" />
+    <xacro:property name="shelf_dist_from_bumper_m" value="0.099475" />
+    <xacro:property name="bumper_to_rail_bottom_offset_z" value="0.1395" />
     <!-- describe the fixed top_shelf to camera_link transform -->
     <xacro:property name="kinect_side_edge_depth_offset_m" value="0.132"/>  <!-- depth lens measured from left edge of top shelf -->

File: config/urdf/shelf.xacro (robot description, xacro)
@@ -12,12 +12,20 @@
     <!-- <xacro:property name="arm_mount_panel_edge_offset_m" value="0.14605" /> -->
     <!-- values measured from husky at lab -->
-    <xacro:property name="shelf_length_m" value="0.126" />
-    <xacro:property name="shelf_width_m" value="0.00700" />
-    <xacro:property name="shelf_height_m" value="0.24324" />
+    <!-- <xacro:property name="shelf_length_m" value="0.126" /> -->
+    <!-- <xacro:property name="shelf_width_m" value="0.00700" /> -->
+    <!-- <xacro:property name="shelf_height_m" value="0.24324" /> -->
+    <!-- <xacro:property name="arm_mount_panel_height_m" value="0.171" /> -->
+    <!-- <xacro:property name="arm_mount_panel_edge_offset_m" value="0.098322" /> -->
+    <!-- <xacro:property name="bottom_shelf_height_offset" value="0.05"/> -->
+    <!-- arm mount panel currently inherits thickness from the shelving unit -->
+    <!-- values measured on 2014-07-08 (and averaged with previous values) -->
+    <xacro:property name="shelf_length_m" value="0.125" />
+    <xacro:property name="shelf_width_m" value="0.00500" />
+    <xacro:property name="shelf_height_m" value="0.24362" />
     <xacro:property name="arm_mount_panel_height_m" value="0.171" />
     <xacro:property name="arm_mount_panel_edge_offset_m" value="0.098322" />
-    <xacro:property name="bottom_shelf_height_offset" value="0.05"/>
+    <xacro:property name="bottom_shelf_height_offset" value="0.045"/>
+    <xacro:property name="top_shelf_length_m" value="0.151"/>
     <!-- arm mount panel currently inherits thickness from the shelving unit -->
-    <xacro:property name="top_shelf_length_m" value="0.151"/>
     <!-- bumper_frame: the name of the frame of the front bumper -->
     <!-- bumper_to_shelf_x: the distance between the bumper frame and the front of the right shelf support -->

Commit message: remeasure kinect model parameters

File: config/urdf/andalite.xacro (robot description, xacro)
@@ -7,4 +7,5 @@
     <include filename="$(find hdt)/config/urdf/shelf.xacro"/>
     <include filename="$(find hdt)/config/urdf/kinect.xacro"/>
+    <!-- describe the fixed front bumper to shelf transforms -->
     <!-- values computed from diagrams -->
     <!-- <xacro:property name="rail_width" value="0.421" />  -->
@@ -19,10 +20,12 @@
     <xacro:property name="shelf_dist_from_bumper_m" value="0.099475" />
     <xacro:property name="bumper_to_rail_bottom_offset_z" value="0.1395" />
-    <!-- describe the fixed top_shelf to camera_link transform -->
-    <xacro:property name="kinect_side_edge_depth_offset_m" value="0.132"/>  <!-- depth lens measured from left edge of top shelf -->
-    <xacro:property name="kinect_front_edge_offset_m" value=".01097"/>      <!-- depth lens measured from front edge of top shelf -->
-    <!-- <xacro:property name="kinect_height_offset_m" value="0.04967"/> -->         <!-- depth lens measured from top edge of top shelf -->
-    <xacro:property name="kinect_height_offset_m" value="0.01"/>         <!-- depth lens measured from top edge of top shelf -->
-    <xacro:property name="kinect_depth_to_camera_offset_ym" value="-0.02"/> <!-- offset from depth lens to camera_link in y -->
+    <!-- describe the fixed top_shelf to kinect_base_link transform -->
+    <!-- <xacro:property name="kinect_side_edge_depth_offset_m" value="0.132"/> -->  <!-- depth lens measured from left edge of top shelf -->
+    <!-- <xacro:property name="kinect_front_edge_offset_m" value=".01097"/> -->      <!-- depth lens measured from front edge of top shelf -->
+    <!-- <xacro:property name="kinect_height_offset_m" value="0.01"/> -->            <!-- depth lens measured from top edge of top shelf -->
+    <!-- <xacro:property name="kinect_depth_to_camera_offset_ym" value="-0.02"/> --> <!-- offset from depth lens to camera_link in y -->
+    <!-- values measured on 2014-07-08 -->
+    <xacro:property name="kinect_side_edge_depth_offset_m" value="0.125"/>
+    <xacro:property name="kinect_front_edge_offset_m" value=".048"/>
     <!-- Build the robot -->
     <xacro:husky_shelf
@@ -33,6 +36,6 @@
     <xacro:kinect
         mounting_link="top_shelf"
-        mounting_origin="${0.5 * shelf_length_m - kinect_front_edge_offset_m}
-                         ${0.5 * rail_width + shelf_width_m - kinect_side_edge_depth_offset_m + kinect_depth_to_camera_offset_ym}
+        mounting_origin="${0.5 * top_shelf_length_m - kinect_front_edge_offset_m}
+                         ${0.5 * rail_width + shelf_width_m - kinect_side_edge_depth_offset_m}
                          ${0.5 * shelf_width_m}"/>
     <xacro:hdt_arm mounting_link="arm_mount_panel_dummy" mounting_origin="0 0 0" />

Commit message: add modified kinect xacro files and replace kinect surrogate with actual kinect meshes and frames

File: config/urdf/andalite.xacro (robot description, xacro)
@@ -7,4 +7,5 @@
     <include filename="$(find hdt)/config/urdf/shelf.xacro"/>
     <include filename="$(find hdt)/config/urdf/kinect.xacro"/>
+    <include filename="$(find hdt)/config/urdf/kinect_camera.urdf.xacro"/>
     <!-- describe the fixed front bumper to shelf transforms -->
     <!-- values computed from diagrams -->
@@ -34,9 +35,15 @@
         bumper_to_shelf_z="${bumper_to_rail_bottom_offset_z}"
         rail_width="${rail_width}"/>
-    <xacro:kinect
-        mounting_link="top_shelf"
-        mounting_origin="${0.5 * top_shelf_length_m - kinect_front_edge_offset_m}
+    <property name="cal_kinect_x" value="0.0"/>
+    <property name="cal_kinect_y" value="0.0"/>
+    <property name="cal_kinect_z" value="0.0"/>
+    <property name="cal_kinect_roll" value="0.0"/>
+    <property name="cal_kinect_pitch" value="0.0"/>
+    <property name="cal_kinect_yaw" value="0.0"/>
+    <xacro:kinect_camera_v0 name="kinect" parent="top_shelf">
+        <origin xyz="${0.5 * top_shelf_length_m - kinect_front_edge_offset_m}
                          ${0.5 * rail_width + shelf_width_m - kinect_side_edge_depth_offset_m}
                          ${0.5 * shelf_width_m}"/>
+    </xacro:kinect_camera_v0>
     <xacro:hdt_arm mounting_link="arm_mount_panel_dummy" mounting_origin="0 0 0" />
     <xacro:fake_gripper mounting_link="arm_7_gripper_lift_link" mounting_origin="${length7+0.075} 0.0 0.0" />

Commit message: correct wrist to gripper transform and make gripper sizes more believable

File: config/urdf/andalite.xacro (robot description, xacro)
@@ -47,4 +47,4 @@
     </xacro:kinect_camera_v0>
     <xacro:hdt_arm mounting_link="arm_mount_panel_dummy" mounting_origin="0 0 0" />
-    <xacro:fake_gripper mounting_link="arm_7_gripper_lift_link" mounting_origin="${length7+0.075} 0.0 0.0" />
+    <xacro:fake_gripper mounting_link="arm_7_gripper_lift_link" mounting_origin="0.062 0.0 0.0" />
 </robot>

File: config/urdf/fake_gripper.xacro (robot description, xacro)
@@ -2,4 +2,12 @@
 <robot xmlns:xacro="http://www.ros.org/wiki/xacro">
     <include filename="$(find hdt)/config/urdf/common.xacro"/>
+    <xacro:property name="gripper_base_length" value="0.084" />
+    <xacro:property name="gripper_base_width" value="0.05" />
+    <xacro:property name="gripper_base_height" value="0.14" />
+    <xacro:property name="finger_span" value="0.0845" />
+    <xacro:property name="finger_length" value="0.07" />
+    <xacro:property name="finger_width" value="${gripper_base_width}" />
+    <!-- <xacro:property name="finger_height" value="${0.5 * (gripper_base_height - finger_span)}" /> -->
+    <xacro:property name="finger_height" value="0.02775" />
     <!-- macro to instantiate the fake gripper -->
     <xacro:macro name="fake_gripper" params="mounting_link mounting_origin">
@@ -13,7 +21,7 @@
             <visual>
                 <geometry>
-                    <box size="0.022 0.140 0.075"/>
+                    <box size="${gripper_base_length} ${gripper_base_width} ${gripper_base_height}"/>
                 </geometry>
-                <origin rpy="${pi/2} 0 ${pi/2}" xyz="${-0.075/2 - 0.03} 0 0"/>
+                <origin xyz="0 0 0" rpy="0 0 0"/>
                 <material name="black">
                     <color rgba="1 1 1 1"/>
@@ -22,7 +30,6 @@
             <collision>
                 <geometry>
-                    <box size="0.022 0.140 0.075"/>
+                    <box size="${gripper_base_length} ${gripper_base_width} ${gripper_base_height}"/>
                 </geometry>
-                <origin rpy="${pi/2} 0 ${pi/2}" xyz="${-0.075/2 - 0.03} 0 0"/>
             </collision>
             <inertial>
@@ -36,5 +43,5 @@
             <limit lower="0.001" upper="0.042" effort="45" velocity="0.38"/>
             <axis xyz="0 0 1"/>
-            <origin xyz="0.0 0.0 0.011"/>
+            <origin xyz="${0.5 * (gripper_base_length + finger_length)} 0 ${0.5 * (gripper_base_height - finger_height)}"/>
             <dynamics damping="10" friction="0.1"/>
         </joint>
@@ -42,14 +49,12 @@
             <visual>
                 <geometry>
-                    <box size="0.022 0.022 0.06"/>
+                    <box size="${finger_length} ${finger_width} ${finger_height}"/>
                 </geometry>
-                <origin rpy="0 ${pi/2} 0" xyz="0.0 0.0 0.00"/>
                 <material name="black"/>
             </visual>
             <collision>
                 <geometry>
-                    <box size="0.022 0.022 0.06"/>
+                    <box size="${finger_length} ${finger_width} ${finger_height}"/>
                 </geometry>
-                <origin rpy="0 ${pi/2} 0" xyz="0.0 0.0 0.00"/>
             </collision>
             <inertial>
@@ -63,5 +68,5 @@
             <limit lower="0.001" upper="0.042" effort="45" velocity="0.38"/>
             <axis xyz="0 0 -1"/>
-            <origin xyz="0.0 0.0 -0.011"/>
+            <origin xyz="${0.5 * (gripper_base_length + finger_length)} 0 ${-0.5 * (gripper_base_height - finger_height)}"/>
             <dynamics damping="10" friction="0.1"/>
         </joint>
@@ -69,14 +74,12 @@
             <visual>
                 <geometry>
-                    <box size="0.022 0.022 0.06"/>
+                    <box size="${finger_length} ${finger_width} ${finger_height}"/>
                 </geometry>
-                <origin rpy="0 ${pi/2} 0" xyz="0.0 0.0 0.00"/>
                 <material name="black"/>
             </visual>
             <collision>
                 <geometry>
-                    <box size="0.022 0.022 0.06"/>
+                    <box size="${finger_length} ${finger_width} ${finger_height}"/>
                 </geometry>
-                <origin rpy="0 ${pi/2} 0" xyz="0.0 0.0 0.00"/>
             </collision>
             <inertial>
