Commit message: some commenting and formatting; fix missing kinect variables

File: config/urdf/andalite.xacro (robot description, xacro)
@@ -6,5 +6,4 @@
     <include filename="$(find hdt)/config/urdf/fake_gripper.xacro"/>
     <include filename="$(find hdt)/config/urdf/shelf.xacro"/>
-    <include filename="$(find hdt)/config/urdf/kinect.xacro"/>
     <include filename="$(find hdt)/config/urdf/kinect_camera.urdf.xacro"/>
     <!-- describe the fixed front bumper to shelf transforms -->

File: config/urdf/kinect.xacro (robot description, xacro)
@@ -1,4 +1,10 @@
 <?xml version="1.0"?>
 <robot xmlns:xacro="http://www.ros.org/wiki/xacro">
+	<!-- Provides:
+		one fixed transform for the base of the kinect
+			kinect_mount
+		one revolute joint for the kinect neck
+			kinect_base_link
+	-->
     <include filename="$(find hdt)/config/urdf/common.xacro"/>
     <xacro:property name="min_tilt_angle" value="${-27 * degrees}"/>

File: config/urdf/kinect_camera.urdf.xacro (robot description, xacro)
@@ -1,104 +1,114 @@
 <?xml version="1.0"?>
-<root xmlns:sensor="http://playerstage.sourceforge.net/gazebo/xmlschema/#sensor"
-      xmlns:controller="http://playerstage.sourceforge.net/gazebo/xmlschema/#controller"
-      xmlns:interface="http://playerstage.sourceforge.net/gazebo/xmlschema/#interface"
-      xmlns:xacro="http://ros.org/wiki/xacro">
-  <!-- Provides:
-       one fixed transform for the base of the kinect
-       one revolute joint for the kinect neck
-       one fixed transform to the canonical frame of the camera
-       multiple fixed transforms for convenient sensor frames -->
-  <include filename="$(find hdt)/config/urdf/kinect_camera.gazebo.xacro" />
-  <xacro:macro name="kinect_camera_v0" params="name parent *origin">
-    <!-- fixed joint from mount link to base link -->
-    <joint name="${name}_mount_joint" type="fixed">
-      <insert_block name="origin" />
-      <parent link="${parent}"/>
-      <child link="${name}_base_link"/>
-    </joint>
-    <!-- revolute tilt joint -->
-    <joint name="${name}_tilt" type="revolute">
-        <parent link="${name}_base_link"/>
-        <child link="${name}_tilt_frame"/>
-        <limit lower="${min_tilt_angle}" upper="${max_tilt_angle}" effort="0.0" velocity="0.0"/>
-        <axis xyz="0 0 1"/>
-        <origin xyz="0.0 0.0 ${1 * inches}" rpy="${pi / 2} 0.0 0.0"/>
-    </joint>
-    <!-- fixed joint from tilt frame to camera frame -->
-    <joint name="${name}_frame_joint" type="fixed">
-      <parent link="${name}_tilt_frame" />
-      <child link="${name}_frame" />
-      <origin xyz="0.03 0.03 0" rpy="${-pi / 2} 0 0" />
-    </joint>
-    <!-- camera frame -> depth frame -->
-    <joint name="${name}_depth_frame_joint" type="fixed">
-      <parent link="${name}_frame" />
-      <child link="${name}_depth_frame" />
-      <origin xyz="0 0.01287 0" />
-    </joint>
-    <!-- camera frame -> rgb frame -->
-    <joint name="${name}_rgb_frame_joint" type="fixed">
-      <parent link="${name}_frame" />
-      <child link="${name}_rgb_frame" />
-      <origin xyz="0 -0.01287 0" />
-    </joint>
-    <!-- depth frame -> depth optical frame -->
-    <joint name="${name}_depth_optical_frame_joint" type="fixed">
-      <parent link="${name}_depth_frame" />
-      <child link="${name}_depth_optical_frame" />
-      <origin xyz="${cal_kinect_x}            ${cal_kinect_y}         ${cal_kinect_z}"
-              rpy="${-M_PI/2+cal_kinect_roll} ${0.0+cal_kinect_pitch} ${-M_PI/2+cal_kinect_yaw}" />
-    </joint>
-    <!-- rgb frame -> rgb optical frame -->
-    <joint name="${name}_rgb_optical_frame_joint" type="fixed">
-      <parent link="${name}_rgb_frame" />
-      <child link="${name}_rgb_optical_frame" />
-      <origin xyz="${cal_kinect_x}            ${cal_kinect_y}         ${cal_kinect_z}"
-              rpy="${-M_PI/2+cal_kinect_roll} ${0.0+cal_kinect_pitch} ${-M_PI/2+cal_kinect_yaw}" />
-    </joint>
-    <!-- base link -->
-    <link name="${name}_base_link">
-        <visual>
-            <geometry>
-                <mesh filename="package://hdt/resource/meshes/kinect_v0/kinect_base.dae" scale="0.001 0.001 0.001"/>
-            </geometry>
-            <origin xyz="0.03 0 0.053" rpy="0 0 0"/>
-        </visual>
-        <collision>
-            <geometry>
-                <mesh filename="package://hdt/resource/meshes/kinect_v0/kinect_base.dae" scale="0.001 0.001 0.001"/>
-            </geometry>
-            <origin xyz="0 0 0.05" rpy="0 0 0"/>
-        </collision>
-    </link>
-    <link name="${name}_tilt_frame" />
-    <!-- camera frame -->
-    <link name="${name}_frame">
-      <inertial>
-        <mass value="0.1" />
-        <origin xyz="0 0 0" rpy="0 0 0"/>
-        <inertia ixx="0.01"  ixy="0.0"  ixz="0.0"
-                 iyy="0.01"  iyz="0.0"
-                 izz="0.01" />
-      </inertial>
-      <visual>
-        <origin xyz="0.0 0.0 0" rpy="0 0 0"/>
-        <geometry>
-          <mesh filename="package://hdt/resource/meshes/kinect_v0/kinect_head.dae" scale="0.001 0.001 0.001" />
-        </geometry>
-      </visual>
-      <collision>
-        <origin xyz="0.0 0.0 0" rpy="0 0 0"/>
-        <geometry>
-          <mesh filename="package://hdt/resource/meshes/kinect_v0/kinect_head.dae" scale="0.001 0.001 0.001" />
-        </geometry>
-      </collision>
-    </link>
-    <link name="${name}_depth_frame" />
-    <link name="${name}_rgb_frame" />
-    <link name="${name}_depth_optical_frame"/>
-    <link name="${name}_rgb_optical_frame"/>
-    <!-- extensions -->
-    <xacro:kinect_camera_gazebo_v0 name="${name}" />
-  </xacro:macro>
+<root xmlns:controller="http://playerstage.sourceforge.net/gazebo/xmlschema/#controller"
+    xmlns:interface="http://playerstage.sourceforge.net/gazebo/xmlschema/#interface"
+    xmlns:sensor="http://playerstage.sourceforge.net/gazebo/xmlschema/#sensor"
+    xmlns:xacro="http://ros.org/wiki/xacro">
+    <!-- Provides:
+        one fixed transform for the base of the kinect:
+            ${name}_mount_joint
+        one revolute joint for the kinect neck:
+            ${name}_tilt one fixed transform to
+        the canonical frame of the camera
+            ${name}_frame_joint
+        multiple fixed transforms for convenient sensor frames:
+            ${name}_depth_frame_joint
+            ${name}_rgb_frame_joint
+            ${name}_depth_optical_frame_joint
+            ${name}_rgb_optical_frame_joint
+    -->
+    <xacro:property name="min_tilt_angle" value="${-27 * degrees}"/>
+    <xacro:property name="max_tilt_angle" value="${ 27 * degrees}"/>
+    <include filename="$(find hdt)/config/urdf/kinect_camera.gazebo.xacro" />
+    <xacro:macro name="kinect_camera_v0" params="name parent *origin">
+        <!-- fixed joint from mount link to base link -->
+        <joint name="${name}_mount_joint" type="fixed">
+            <insert_block name="origin" />
+            <parent link="${parent}"/>
+            <child link="${name}_base_link"/>
+        </joint>
+        <!-- revolute tilt joint -->
+        <joint name="${name}_tilt" type="revolute">
+            <parent link="${name}_base_link"/>
+            <child link="${name}_tilt_frame"/>
+            <limit lower="${min_tilt_angle}" upper="${max_tilt_angle}" effort="0.0" velocity="0.0"/>
+            <axis xyz="0 0 1"/>
+            <origin xyz="0.0 0.0 ${1 * inches}" rpy="${pi / 2} 0.0 0.0"/>
+        </joint>
+        <!-- fixed joint from tilt frame to camera frame -->
+        <joint name="${name}_frame_joint" type="fixed">
+            <parent link="${name}_tilt_frame" />
+            <child link="${name}_frame" />
+            <origin xyz="0.03 0.03 0" rpy="${-pi / 2} 0 0" />
+        </joint>
+        <!-- camera frame -> depth frame -->
+        <joint name="${name}_depth_frame_joint" type="fixed">
+            <parent link="${name}_frame" />
+            <child link="${name}_depth_frame" />
+            <origin xyz="0 0.01287 0" />
+        </joint>
+        <!-- camera frame -> rgb frame -->
+        <joint name="${name}_rgb_frame_joint" type="fixed">
+            <parent link="${name}_frame" />
+            <child link="${name}_rgb_frame" />
+            <origin xyz="0 -0.01287 0" />
+        </joint>
+        <!-- depth frame -> depth optical frame -->
+        <joint name="${name}_depth_optical_frame_joint" type="fixed">
+            <parent link="${name}_depth_frame" />
+            <child link="${name}_depth_optical_frame" />
+            <origin xyz="${cal_kinect_x} ${cal_kinect_y} ${cal_kinect_z}"
+                    rpy="${-M_PI/2+cal_kinect_roll} ${0.0+cal_kinect_pitch} ${-M_PI/2+cal_kinect_yaw}" />
+        </joint>
+        <!-- rgb frame -> rgb optical frame -->
+        <joint name="${name}_rgb_optical_frame_joint" type="fixed">
+            <parent link="${name}_rgb_frame" />
+            <child link="${name}_rgb_optical_frame" />
+            <origin xyz="${cal_kinect_x} ${cal_kinect_y} ${cal_kinect_z}"
+                    rpy="${-M_PI/2+cal_kinect_roll} ${0.0+cal_kinect_pitch} ${-M_PI/2+cal_kinect_yaw}" />
+        </joint>
+        <!-- base link -->
+        <link name="${name}_base_link">
+            <visual>
+                <geometry>
+                    <mesh filename="package://hdt/resource/meshes/kinect_v0/kinect_base.dae" scale="0.001 0.001 0.001"/>
+                </geometry>
+                <origin xyz="0.03 0 0.053" rpy="0 0 0"/>
+            </visual>
+            <collision>
+                <geometry>
+                    <mesh filename="package://hdt/resource/meshes/kinect_v0/kinect_base.dae" scale="0.001 0.001 0.001"/>
+                </geometry>
+                <origin xyz="0 0 0.05" rpy="0 0 0"/>
+            </collision>
+        </link>
+        <link name="${name}_tilt_frame" />
+        <!-- camera frame -->
+        <link name="${name}_frame">
+            <inertial>
+                <mass value="0.1" />
+                <origin xyz="0 0 0" rpy="0 0 0"/>
+                <inertia ixx="0.01" ixy="0.0" ixz="0.0" iyy="0.01" iyz="0.0" izz="0.01" />
+            </inertial>
+            <visual>
+                <origin xyz="0.0 0.0 0" rpy="0 0 0"/>
+                <geometry>
+                    <mesh filename="package://hdt/resource/meshes/kinect_v0/kinect_head.dae" scale="0.001
+                        0.001 0.001" />
+                </geometry>
+            </visual>
+            <collision>
+                <origin xyz="0.0 0.0 0" rpy="0 0 0"/>
+                <geometry>
+                    <mesh filename="package://hdt/resource/meshes/kinect_v0/kinect_head.dae" scale="0.001
+                        0.001 0.001" />
+                </geometry>
+            </collision>
+        </link>
+        <link name="${name}_depth_frame" />
+        <link name="${name}_rgb_frame" />
+        <link name="${name}_depth_optical_frame"/>
+        <link name="${name}_rgb_optical_frame"/>
+        <!-- extensions -->
+        <xacro:kinect_camera_gazebo_v0 name="${name}" />
+    </xacro:macro>
 </root>
