Commit message: correct top shelf height and add parameter to describe top shelf overhang

File: config/urdf/shelf.xacro (robot description, xacro)
@@ -17,6 +17,7 @@
     <xacro:property name="arm_mount_panel_height_m" value="0.171" />
     <xacro:property name="arm_mount_panel_edge_offset_m" value="0.098322" />
+    <xacro:property name="bottom_shelf_height_offset" value="0.05"/>
     <!-- arm mount panel currently inherits thickness from the shelving unit -->
-    <xacro:property name="bottom_shelf_height_offset" value="0.05"/>
+    <xacro:property name="top_shelf_length_m" value="0.151"/>
     <!-- bumper_frame: the name of the frame of the front bumper -->
     <!-- bumper_to_shelf_x: the distance between the bumper frame and the front of the right shelf support -->
@@ -49,5 +50,5 @@
             <parent link="${bumper_frame}" />
             <child link="top_shelf" />
-            <origin xyz="${-bumper_to_shelf_x - 0.5 * shelf_length_m} 0.0 ${bumper_to_shelf_z + shelf_height_m - 0.5 * shelf_width_m}"
+            <origin xyz="${-bumper_to_shelf_x - shelf_length_m + 0.5 * top_shelf_length_m} 0.0 ${bumper_to_shelf_z + shelf_height_m + 0.5 * shelf_width_m}"
                     rpy="0 0 0" />
         </joint>
@@ -104,5 +105,5 @@
             <visual>
                 <geometry>
-                    <box size="${shelf_length_m} ${rail_width + 2 * shelf_width_m} ${shelf_width_m}" />
+                    <box size="${top_shelf_length_m} ${rail_width + 2 * shelf_width_m} ${shelf_width_m}" />
                 </geometry>
                 <material name="gray">
@@ -112,5 +113,5 @@
             <collision>
                 <geometry>
-                    <box size="${shelf_length_m} ${rail_width} ${shelf_width_m}" />
+                    <box size="${top_shelf_length_m} ${rail_width + 2 * shelf_width_m} ${shelf_width_m}" />
                 </geometry>
             </collision>

Commit message: update arm mount panel location in urdf (moved after mounting asus)

File: config/urdf/shelf.xacro (robot description, xacro)
@@ -24,8 +24,10 @@
     <xacro:property name="shelf_height_m" value="0.24362" />
     <xacro:property name="arm_mount_panel_height_m" value="0.171" />
-    <xacro:property name="arm_mount_panel_edge_offset_m" value="0.098322" />
+    <!-- <xacro:property name="arm_mount_panel_edge_offset_m" value="0.098322" /> -->
     <xacro:property name="bottom_shelf_height_offset" value="0.045"/>
     <xacro:property name="top_shelf_length_m" value="0.151"/>
     <!-- arm mount panel currently inherits thickness from the shelving unit -->
+    <!-- values measure on 2014-08-07 (moved arm mount due to no room to mount asus servo) -->
+    <xacro:property name="arm_mount_panel_edge_offset_m" value="0.07508" />
     <!-- bumper_frame: the name of the frame of the front bumper -->
     <!-- bumper_to_shelf_x: the distance between the bumper frame and the front of the right shelf support -->
