Commit message: initial modeling of tilt mount, working in sim and pending live measurement data

File: config/urdf/andalite_with_asus.xacro (robot description, xacro)
@@ -7,4 +7,5 @@
     <include filename="$(find hdt)/config/urdf/shelf.xacro"/>
     <include filename="$(find hdt)/config/urdf/asus_camera.urdf.xacro"/>
+    <include filename="$(find hdt)/config/urdf/tilt_mount.xacro"/>
     <!-- describe the fixed front bumper to shelf transforms -->
     <!-- values computed from diagrams -->
@@ -45,8 +46,11 @@
     <xacro:property name="asus_bay_top_offset_m" value="0.110"/>            <!-- The top of the housing surrounding the camera from the top of the top shelf -->
     <xacro:property name="asus_bay_bottom_offset_m" value="0.145"/>         <!-- The bottom of the housing surrounding the camera from the top of the top shelf -->
-    <xacro:asus_xtion_pro_live name="asus" parent="top_shelf">
-        <origin xyz="${0.5 * top_shelf_length_m}
+    <xacro:tilt_mount name="tilt_mount" parent="top_shelf">
+        <origin xyz="0
                      ${0.5 * rail_width + shelf_width_m - 0.5 * (asus_left_screw_mount_offset_m + asus_right_screw_mount_offset_m)}
-                     ${0.5 * shelf_width_m - 0.5 * (asus_bay_top_offset_m + asus_bay_bottom_offset_m)}"/>
+                     ${-0.5 * shelf_width_m}"/>
+    </xacro:tilt_mount>
+    <xacro:asus_xtion_pro_live name="asus" parent="tilt_mount_sensor_basket">
+        <origin xyz="0.05 ${-0.5 * basket_part_ab_width_m - basket_part_c_width_m - 0.5 * 0.035} 0" rpy="${-pi / 2} 0 0"/>
     </xacro:asus_xtion_pro_live>
     <xacro:hdt_arm mounting_link="arm_mount_panel_dummy" mounting_origin="0 0 0" />

File: config/urdf/asus_camera.urdf.xacro (robot description, xacro)
@@ -22,7 +22,8 @@
             <insert_block name="origin" />
             <parent link="${parent}"/>
-            <child link="${name}_base_link"/>
+            <child link="${name}_frame"/>
         </joint>
         <!-- fixed joint from tilt frame to camera frame -->
+        <!--
         <joint name="${name}_frame_joint" type="fixed">
             <parent link="${name}_base_link" />
@@ -30,4 +31,5 @@
             <origin xyz="0.0 0.0 0" rpy="0 0 0" />
         </joint>
+        -->
         <!-- camera frame -> depth frame -->
         <joint name="${name}_depth_frame_joint" type="fixed">
@@ -57,5 +59,5 @@
         </joint>
         <!-- base link -->
-        <link name="${name}_base_link" />
+        <!-- <link name="${name}_base_link" /> -->
         <!-- camera frame -->
         <link name="${name}_frame">

File: config/urdf/kinect_camera.urdf.xacro (robot description, xacro)
@@ -1,7 +1,7 @@
 <?xml version="1.0"?>
-<root xmlns:controller="http://playerstage.sourceforge.net/gazebo/xmlschema/#controller"
-    xmlns:interface="http://playerstage.sourceforge.net/gazebo/xmlschema/#interface"
-    xmlns:sensor="http://playerstage.sourceforge.net/gazebo/xmlschema/#sensor"
-    xmlns:xacro="http://ros.org/wiki/xacro">
+<robot xmlns:controller="http://playerstage.sourceforge.net/gazebo/xmlschema/#controller"
+       xmlns:interface="http://playerstage.sourceforge.net/gazebo/xmlschema/#interface"
+       xmlns:sensor="http://playerstage.sourceforge.net/gazebo/xmlschema/#sensor"
+       xmlns:xacro="http://ros.org/wiki/xacro">
     <!-- Provides:
         one fixed transform for the base of the kinect:
