Commit message: remove intermediate asus base frame; fill tilt mount dimensions from live measurements; fix up live urdf with asus

File: config/urdf/andalite_no_asus.xacro (robot description, xacro)
@@ -6,4 +6,5 @@
     <include filename="$(find hdt)/config/urdf/fake_gripper.xacro"/>
     <include filename="$(find hdt)/config/urdf/shelf.xacro"/>
+    <include filename="$(find hdt)/config/urdf/tilt_mount.xacro"/>
     <include filename="$(find hdt)/config/urdf/asus.xacro"/>
     <!-- describe the fixed front bumper to shelf transforms -->
@@ -42,8 +43,14 @@
     <property name="cal_kinect_pitch" value="0.0"/>
     <property name="cal_kinect_yaw" value="0.0"/>
-    <xacro:asus_xtion_pro_live name="asus" parent="top_shelf">
-        <origin xyz="${0.5 * top_shelf_length_m}
+    <xacro:tilt_mount name="tilt_mount" parent="top_shelf">
+        <origin xyz="${0.5 * top_shelf_length_m - 0.5 * cradle_part_a_length_m}
                      ${0.5 * rail_width + shelf_width_m - 0.5 * (asus_left_screw_mount_offset_m + asus_right_screw_mount_offset_m)}
-                     ${0.5 * shelf_width_m - 0.5 * (asus_bay_top_offset_m + asus_bay_bottom_offset_m)}"/>
+                     ${-0.5 * shelf_width_m}"/>
+    </xacro:tilt_mount>
+    <xacro:asus_xtion_pro_live name="asus" parent="tilt_mount_sensor_basket">
+        <origin xyz="${0.5 * basket_part_c_length_m}
+                    ${-0.5 * basket_part_ab_width_m - basket_part_c_width_m - 0.5 * basket_sensor_gap}
+                    0"
+                rpy="${-pi / 2} 0 0"/>
     </xacro:asus_xtion_pro_live>
     <xacro:hdt_arm mounting_link="arm_mount_panel_dummy" mounting_origin="0 0 0" />

File: config/urdf/andalite_with_asus.xacro (robot description, xacro)
@@ -29,4 +29,9 @@
     <xacro:property name="kinect_side_edge_depth_offset_m" value="0.125"/>
     <xacro:property name="kinect_front_edge_offset_m" value=".048"/>
+    <!-- values measured on 2014-07-08 -->
+    <xacro:property name="asus_left_screw_mount_offset_m" value="0.242"/>   <!-- The left side of the left screw (facing the robot) from the right edge of the top shelf -->
+    <xacro:property name="asus_right_screw_mount_offset_m" value="0.114"/>  <!-- The left side of the right screw (facing the robot) from the right edge of the top shelf -->
+    <xacro:property name="asus_bay_top_offset_m" value="0.110"/>            <!-- The top of the housing surrounding the camera from the top of the top shelf -->
+    <xacro:property name="asus_bay_bottom_offset_m" value="0.145"/>         <!-- The bottom of the housing surrounding the camera from the top of the top shelf -->
     <!-- Build the robot -->
     <xacro:husky_shelf
@@ -41,9 +46,4 @@
     <property name="cal_kinect_pitch" value="0.0"/>
     <property name="cal_kinect_yaw" value="0.0"/>
-    <!-- values measured on 2014-07-08 -->
-    <xacro:property name="asus_left_screw_mount_offset_m" value="0.242"/>   <!-- The left side of the left screw (facing the robot) from the right edge of the top shelf -->
-    <xacro:property name="asus_right_screw_mount_offset_m" value="0.114"/>  <!-- The left side of the right screw (facing the robot) from the right edge of the top shelf -->
-    <xacro:property name="asus_bay_top_offset_m" value="0.110"/>            <!-- The top of the housing surrounding the camera from the top of the top shelf -->
-    <xacro:property name="asus_bay_bottom_offset_m" value="0.145"/>         <!-- The bottom of the housing surrounding the camera from the top of the top shelf -->
     <xacro:tilt_mount name="tilt_mount" parent="top_shelf">
         <origin xyz="0

File: config/urdf/asus.xacro (robot description, xacro)
@@ -1,7 +1,9 @@
 <?xml version="1.0"?>
 <robot xmlns:xacro="http://ros.org/wiki/xacro">
-    <!-- Provides:
-         one fixed transform for the base of the asus
-         one fixed transform -->
+    <!--
+    Provides:
+         a canonical camera frame
+         one fixed transform from the mounting frame to the camera frame
+    -->
     <xacro:macro name="asus_xtion_pro_live" params="name parent *origin">
         <!-- fixed transform for the base of the asus -->
@@ -9,14 +11,7 @@
             <insert_block name="origin"/>
             <parent link="${parent}"/>
-            <child link="${name}_base_link"/>
+            <child link="${name}_link"/>
         </joint>
-        <!-- fixed transform from the camera base frame to the canonical camera frame -->
-        <joint name="${name}_frame_joint" type="fixed">
-            <parent link="${name}_base_link"/>
-            <child link="${name}_link"/>
-            <origin xyz="0 0 0" rpy="0 0 0"/>
-        </joint>
-        <!-- dummy link for offset from mounting link and canonical camera frame -->
-        <link name="${name}_base_link"/>
+        <!-- canonical frame of the camera -->
         <link name="${name}_link"/>
     </xacro:macro>

File: config/urdf/tilt_mount.xacro (robot description, xacro)
@@ -1,30 +1,36 @@
 <?xml version="1.0"?>
 <robot xmlns:xacro="http://www.ros.org/wiki/xacro">
-    <xacro:property name="plate_thickness_m" value="0.0116667"/>
-    <xacro:property name="plate_length_m" value="0.10"/>
+    <!-- values measured on 2014-08-27 -->
     <!-- cradle properties -->
-    <xacro:property name="cradle_part_a_length_m" value="0.10"/> <!-- plate_length_m -->
-    <xacro:property name="cradle_part_a_width_m" value="0.256"/>
-    <xacro:property name="cradle_part_a_height_m" value="0.0116667"/> <!-- plate_thickness_m -->
-    <xacro:property name="cradle_part_bc_length_m" value="0.10"/> <!-- plate_length_m -->
-    <xacro:property name="cradle_part_bc_width_m" value="0.123"/>
-    <xacro:property name="cradle_part_bc_height_m" value="0.0116667"/> <!-- plate_thickness_m -->
-    <xacro:property name="cradle_part_de_length_m" value="0.10"/> <!-- plate_length_m -->
-    <xacro:property name="cradle_part_de_width_m" value="0.0116667"/> <!-- plate_thickness_m -->
-    <xacro:property name="cradle_part_de_height_m" value="0.1113333"/>
-    <xacro:property name="servo_length_m" value="0.10"/>
-    <xacro:property name="servo_width_m" value="0.0556665"/>
-    <xacro:property name="servo_height_m" value="0.08349975"/>
+    <xacro:property name="cradle_part_a_length_m" value="0.04077"/>
+    <xacro:property name="cradle_part_a_width_m" value="0.25419"/>
+    <xacro:property name="cradle_part_a_height_m" value="0.0122"/>
+    <!-- the distance that parts a and b hang off the edge of part a -->
+    <xacro:property name="cradle_abc_offset_m" value="0.01070"/>
+    <xacro:property name="cradle_part_bc_length_m" value="0.04077"/>
+    <xacro:property name="cradle_part_bc_width_m" value="0.09384"/>
+    <xacro:property name="cradle_part_bc_height_m" value="0.00630"/>
+    <xacro:property name="cradle_part_de_length_m" value="0.04077"/>
+    <xacro:property name="cradle_part_de_width_m" value="0.00630"/>
+    <xacro:property name="cradle_part_de_height_m" value="0.07745"/>
+    <xacro:property name="servo_length_m" value="0.04077"/>
+    <xacro:property name="servo_width_m" value="0.043305"/>
+    <xacro:property name="servo_height_m" value="0.069275"/>
+    <!-- properties for determining the revolute joint origin -->
+    <!-- the distance from the bottom of the servo to the center of the hinge -->
+    <xacro:property name="servo_hinge_offset_m" value="0.01426"/>
+    <!-- the distance from the bottom of parts a and b to the center of the screw/hinge -->
+    <xacro:property name="basket_ab_hinge_offset_m" value="0.02857"/>
     <!-- basket properties -->
-    <xacro:property name="basket_part_ab_length_m" value="0.10"/> <!-- plate_length_m -->
-    <xacro:property name="basket_part_ab_width_m" value="0.065"/>
-    <xacro:property name="basket_part_ab_height_m" value="0.0116667"/>
-    <xacro:property name="basket_part_c_length_m" value="0.10"/> <!-- plate_length_m -->
-    <xacro:property name="basket_part_c_width_m" value="0.0116667"/>
-    <xacro:property name="basket_part_c_height_m" value="0.25"/>
-    <xacro:property name="basket_sensor_gap" value="0.035"/>
-    <xacro:property name="basket_part_d_length_m" value="0.10"/> <!-- plate_length_m -->
-    <xacro:property name="basket_part_d_width_m" value="0.0116667"/>
-    <xacro:property name="basket_part_d_height_m" value="0.23"/>
+    <xacro:property name="basket_part_ab_length_m" value="0.0598"/>
+    <xacro:property name="basket_part_ab_width_m" value="0.05477"/>
+    <xacro:property name="basket_part_ab_height_m" value="0.0066"/>
+    <xacro:property name="basket_part_c_length_m" value="0.0598"/>
+    <xacro:property name="basket_part_c_width_m" value="0.00654"/>
+    <xacro:property name="basket_part_c_height_m" value="0.22885"/>
+    <xacro:property name="basket_sensor_gap" value="0.0203"/>
+    <xacro:property name="basket_part_d_length_m" value="0.01907"/>
+    <xacro:property name="basket_part_d_width_m" value="0.00953"/>
+    <xacro:property name="basket_part_d_height_m" value="0.20599"/>
     <material name="gray">
         <color rgba="0.5 0.5 0.5 1.0"/>
@@ -41,7 +47,7 @@
             <parent link="${name}_servo_cradle"/>
             <child link="${name}_sensor_basket"/>
-            <limit lower="${-30 * degrees}" upper="${30 * degrees}" effort="0.0" velocity="0.0"/>
+            <limit lower="${-30 * degrees}" upper="${30 * degrees}" effort="0.0" velocity="0.0"/> <!-- dummy limits -->
             <axis xyz="0 0 1"/>
-            <origin xyz="0.0 0.0 -0.08" rpy="${pi / 2} 0.0 0.0"/>
+            <origin xyz="0.0 0.0 ${-(cradle_part_a_height_m + cradle_part_bc_height_m + servo_height_m - servo_hinge_offset_m + basket_ab_hinge_offset_m - 0.5 * basket_part_ab_width_m)}" rpy="${pi / 2} 0.0 0.0"/>
         </joint>
         <link name="${name}_servo_cradle">
@@ -60,5 +66,5 @@
             <visual name="part_b">
                 <origin xyz="0
-                             ${ 0.167 * cradle_part_a_width_m + 0.5 * cradle_part_bc_width_m}
+                             ${-0.5 * cradle_part_a_width_m - cradle_abc_offset_m + 0.5 * cradle_part_bc_width_m}
                              ${-cradle_part_a_height_m - 0.5 * cradle_part_bc_height_m}"/>
                 <geometry>
@@ -69,5 +75,5 @@
             <visual name="part_c">
                 <origin xyz="0
-                             ${-0.167 * cradle_part_a_width_m - 0.5 * cradle_part_bc_width_m}
+                             ${ 0.5 * cradle_part_a_width_m + cradle_abc_offset_m - 0.5 * cradle_part_bc_width_m}
                              ${-cradle_part_a_height_m - 0.5 * cradle_part_bc_height_m}"/>
                 <geometry>
@@ -78,5 +84,5 @@
             <visual name="part_d">
                 <origin xyz="0
-                             ${ 0.167 * cradle_part_a_width_m + cradle_part_bc_width_m - 0.5 * cradle_part_de_width_m}
+                             ${-0.5 * cradle_part_a_width_m - cradle_abc_offset_m + 0.5 * cradle_part_de_width_m}
                              ${-cradle_part_a_height_m - cradle_part_bc_height_m - 0.5 * cradle_part_de_height_m}"/>
                 <geometry>
@@ -87,5 +93,5 @@
             <visual name="part_e">
                 <origin xyz="0
-                             ${-0.167 * cradle_part_a_width_m - cradle_part_bc_width_m + 0.5 * cradle_part_de_width_m}
+                             ${ 0.5 * cradle_part_a_width_m + cradle_abc_offset_m - 0.5 * cradle_part_de_width_m}
                              ${-cradle_part_a_height_m - cradle_part_bc_height_m - 0.5 * cradle_part_de_height_m}"/>
                 <geometry>
@@ -96,5 +102,5 @@
             <visual name="right_servo">
                 <origin xyz="0
-                             ${+0.167 * cradle_part_a_width_m + cradle_part_bc_width_m - cradle_part_de_width_m - 0.5 * servo_width_m}
+                             ${-0.5 * cradle_part_a_width_m - cradle_abc_offset_m + cradle_part_de_width_m + 0.5 * servo_width_m}
                              ${-cradle_part_a_height_m - cradle_part_bc_height_m - 0.5 * servo_height_m}"/>
                 <geometry>
@@ -105,5 +111,5 @@
             <visual name="left_servo">
                 <origin xyz="0
-                             ${-0.167 * cradle_part_a_width_m - cradle_part_bc_width_m + cradle_part_de_width_m + 0.5 * servo_width_m}
+                             ${ 0.5 * cradle_part_a_width_m + cradle_abc_offset_m - cradle_part_de_width_m - 0.5 * servo_width_m}
                              ${-cradle_part_a_height_m - cradle_part_bc_height_m - 0.5 * servo_height_m}"/>
                 <geometry>
@@ -141,5 +147,7 @@
             <!-- part d -->
             <visual name="part_d">
-                <origin xyz="0 ${-0.5 * basket_part_ab_width_m - basket_part_c_width_m - basket_sensor_gap - 0.5 * basket_part_d_width_m} 0"/>
+                <origin xyz="${0.5 * basket_part_c_length_m - 0.5 * basket_part_d_length_m}
+                             ${-0.5 * basket_part_ab_width_m - basket_part_c_width_m - basket_sensor_gap - 0.5 * basket_part_d_width_m}
+                             0"/>
                 <geometry>
                     <box size="${basket_part_d_length_m} ${basket_part_d_width_m} ${basket_part_d_height_m}"/>
