Commit message: regenerate flubbed up kinematics
Former-commit-id: 141684dac864922fb754507cfe1ca4ee5e6e3cda

File: config/urdf/hdt2.xacro (robot description, xacro)
@@ -150,5 +150,5 @@
             <child link="arm_5_wrist_twist_link"/>
             <!-- <limit lower="${-90*degrees}" upper="${90*degrees}" effort="10" velocity="0.38"/> -->
-            <limit lower="${-30*degrees}" upper="${15*degrees}" effort="10" velocity="0.38"/>
+            <limit lower="${-85*degrees}" upper="${85*degrees}" effort="10" velocity="0.38"/>
             <safety_controller soft_lower_limit="${-85*degrees}" soft_upper_limit="${85*degrees}" k_velocity="0" />
             <axis xyz="0 0 1"/>
