Commit message: attach robotiq 3 finger grippers to roman urdf
Former-commit-id: 28a2dacd8d4085d9cb3f2e1ca532c9ce63f38405

File: src/roman_model/urdf/robosimian_l_arm.urdf.xacro (robot description, xacro)
@@ -3,4 +3,5 @@
     <xacro:include filename="$(find roman_model)/gazebo/robosimian_l_arm.gazebo.xacro"/>
     <xacro:include filename="$(find roman_model)/control/robosimian_l_arm.transmission.xacro"/>
+    <xacro:include filename="$(find robotiq_s_model_visualization)/cfg/s-model_articulated_macro.xacro"/>
     <xacro:macro name="robosimian_l_arm" params="name parent *origin namespace">
         <link name="limb_left_link0">
@@ -183,16 +184,16 @@
             </inertial>
             <visual>
-                <origin xyz="0.087500 0 0" rpy="0 3.141593 -1.570796"/>
-                <geometry>
-                    <box size="0.13 0.13 0.11"/>
-                </geometry>
-                <material name="grey">
-                    <color rgba="0.8 0.8 0.8 1"/>
-                </material>
-            </visual>
-            <collision>
-                <origin rpy="3.1415 -1.57080 0" xyz="0.0875 0 0"/>
-                <geometry>
-                    <box size="0.13 0.13 0.11"/>
+                <origin xyz="0.03016 -0.004 0" rpy="0 1.57080 0"/>
+                <geometry>
+                    <cylinder radius="0.05285" length="0.06032"/>
+                </geometry>
+                <material name="grey">
+                    <color rgba="0.8 0.8 0.8 1"/>
+                </material>
+            </visual>
+            <collision>
+                <origin xyz="0.03016 -0.004 0" rpy="0 1.57080 0"/>
+                <geometry>
+                    <cylinder radius="0.05285" length="0.06032"/>
                 </geometry>
             </collision>
@@ -262,4 +263,12 @@
             <dynamics damping="1.0" friction="10"/>
         </joint>
+        <xacro:s-model_articulated prefix="limb_left_"/>
+        <!-- attach the robotiq gripper to the arm -->
+        <joint name="limb_left_palm_joint" type="fixed">
+            <origin xyz="0.104775 -0.004 0" rpy="3.1415 0 1.57080"/>
+            <axis xyz="0 0 1"/>
+            <parent link="limb_left_link7"/>
+            <child link="limb_left_palm"/>
+        </joint>
         <xacro:robosimian_l_arm_gazebo name="${name}" namespace="${namespace}"/>
         <xacro:robosimian_l_arm_transmission name="${name}" namespace="${namespace}"/>

File: src/roman_model/urdf/robosimian_r_arm.urdf.xacro (robot description, xacro)
@@ -3,4 +3,5 @@
     <xacro:include filename="$(find roman_model)/gazebo/robosimian_r_arm.gazebo.xacro"/>
     <xacro:include filename="$(find roman_model)/control/robosimian_r_arm.transmission.xacro"/>
+    <xacro:include filename="$(find robotiq_s_model_visualization)/cfg/s-model_articulated_macro.xacro"/>
     <xacro:macro name="robosimian_r_arm" params="name parent *origin namespace">
         <link name="limb_right_link0">
@@ -183,16 +184,16 @@
             </inertial>
             <visual>
-                <origin xyz="0.087500 0 0" rpy="0 3.141593 -1.570796"/>
-                <geometry>
-                    <box size="0.13 0.13 0.11"/>
-                </geometry>
-                <material name="grey">
-                    <color rgba="0.8 0.8 0.8 1"/>
-                </material>
-            </visual>
-            <collision>
-                <origin rpy="3.1415 -1.5708 0" xyz="0.0875 0 0"/>
-                <geometry>
-                    <box size="0.13 0.13 0.11"/>
+                <origin xyz="0.03016 -0.004 0" rpy="0 1.57080 0"/>
+                <geometry>
+                    <cylinder radius="0.05285" length="0.06032"/>
+                </geometry>
+                <material name="grey">
+                    <color rgba="0.8 0.8 0.8 1"/>
+                </material>
+            </visual>
+            <collision>
+                <origin xyz="0.03016 -0.004 0" rpy="0 1.57080 0"/>
+                <geometry>
+                    <cylinder radius="0.05285" length="0.06032"/>
                 </geometry>
             </collision>
@@ -262,4 +263,11 @@
             <dynamics damping="1.0" friction="10"/>
         </joint>
+        <xacro:s-model_articulated prefix="limb_right_"/>
+        <joint name="limb_right_palm_joint" type="fixed">
+            <origin xyz="0.104775 -0.004 0" rpy="3.1415 0 1.57080"/>
+            <axis xyz="0 0 1"/>
+            <parent link="limb_right_link7"/>
+            <child link="limb_right_palm"/>
+        </joint>
         <xacro:robosimian_r_arm_gazebo name="${name}" namespace="${namespace}"/>
         <xacro:robosimian_r_arm_transmission name="${name}" namespace="${namespace}"/>
