Commit message: remove zero volume collision objects from roman urdf
Former-commit-id: 37d06364ed7a7e7f84f151ceea239c4ce22391ee

File: src/roman_model/urdf/talon.urdf.xacro (robot description, xacro)
@@ -4,21 +4,5 @@
     <xacro:include filename="$(find roman_model)/control/talon.transmission.xacro"/>
     <xacro:macro name="talon" params="name namespace">
-        <link name="${name}_link">
-            <visual>
-                <origin xyz="0 0 0" rpy="0 0 0"/>
-                <geometry>
-                    <box size="0 0 0"/>
-                </geometry>
-                <material name="white">
-                    <color rgba="1 1 1 1"/>
-                </material>
-            </visual>
-            <collision>
-                <origin rpy="0 0 0" xyz="0 0 0"/>
-                <geometry>
-                    <box size="0 0 0"/>
-                </geometry>
-            </collision>
-        </link>
+        <link name="${name}_link"/>
         <joint name="${name}_joint" type="fixed">
             <origin xyz="0 0 0" rpy="3.14 0 0"/>
@@ -39,5 +23,5 @@
                 </geometry>
                 <material name="grey">
-                    <color rgba=".8 .8 .8 1"/>
+                    <color rgba="0.8 0.8 0.8 1"/>
                 </material>
             </visual>
@@ -69,5 +53,5 @@
         <link name="track_left">
             <inertial>
-                <mass value="0.000000" />
+                <mass value="0.000000"/>
                 <origin xyz="0.000000 0.000000 0.000000" rpy="0 0 0"/>
                 <inertia ixx="0.000000" ixy="0.000000" ixz="0.000000" iyy="0.000000" iyz="0.000000" izz="0.000000"/>

Commit message: add base_footprint joint to roman
Former-commit-id: d5a71d2699a3f47446f3cdce83929e74702177ba

File: src/roman_model/urdf/talon.urdf.xacro (robot description, xacro)
@@ -4,4 +4,10 @@
     <xacro:include filename="$(find roman_model)/control/talon.transmission.xacro"/>
     <xacro:macro name="talon" params="name namespace">
+        <link name="${name}_footprint"/>
+        <joint name="${name}_footprint_joint" type="fixed">
+            <origin xyz="0 0 0.15203" rpy="0 0 0"/>
+            <parent link="${name}_footprint"/>
+            <child link="${name}_link"/>
+        </joint>
         <link name="${name}_link"/>
         <joint name="${name}_joint" type="fixed">

Commit message: replace talon mesh with new version; add surrogate hokuyo to base urdf
Former-commit-id: 61e973e0c3c354df8ecb64c2ecc5fa08a07d3030

File: src/roman_model/urdf/talon.urdf.xacro (robot description, xacro)
@@ -3,4 +3,5 @@
     <xacro:include filename="$(find roman_model)/gazebo/talon.gazebo.xacro"/>
     <xacro:include filename="$(find roman_model)/control/talon.transmission.xacro"/>
+    <xacro:include filename="$(find hector_sensors_description)/urdf/hokuyo_utm30lx.urdf.xacro"/>
     <xacro:macro name="talon" params="name namespace">
         <link name="${name}_footprint"/>
@@ -28,5 +29,5 @@
                 <geometry>
 <!--                    <box size="0.9 0.6 0.26"/> -->
-                    <mesh filename="package://roman_model/meshes/talon.stl" scale="1 1 1"/>
+                    <mesh filename="package://roman_model/meshes/tl1.stl" scale="1 1 1"/>
                 </geometry>
                 <material name="grey">
@@ -63,4 +64,7 @@
             </collision>
         </link>
+        <xacro:hokuyo_utm30lx_gpu name="base_laser" parent="base_link" ros_topic="base_scan" update_rate="20.0" ray_count="1080" min_angle="-130" max_angle="130">
+            <origin xyz="0.413 0 0.210" rpy="0 0 0"/>
+        </xacro:hokuyo_utm30lx_gpu>
         <joint name="track_left_joint" type="revolute">
             <origin xyz="0 0 0" rpy="0 0 0"/>

Commit message: update talon collision model
Former-commit-id: b9634521b56091c6405724fe5d3065fc1a77c9ae

File: src/roman_model/urdf/talon.urdf.xacro (robot description, xacro)
@@ -39,26 +39,26 @@
                 <origin xyz="0 0 0" rpy="0 0 0"/>
                 <geometry>
-                    <box size="0.9 0.6 0.26"/>
+                    <box size="1.070000 0.645000 0.305000"/>
                 </geometry>
             </collision>
             <!-- left track -->
             <collision>
-                <origin xyz="0 0.26 0" rpy="0 0 0"/>
+                <origin xyz="0.000000 0.260000 0.000000" rpy="0 0 0"/>
                 <geometry>
-                    <box size="0.9 0.08 0.3"/>
+                    <box size="1.070000 0.080000 0.300000"/>
                 </geometry>
             </collision>
             <!-- right track -->
             <collision>
-                <origin xyz="0 -0.26 0" rpy="0 0 0"/>
+                <origin xyz="0.000000 -0.260000 0.000000" rpy="0 0 0"/>
                 <geometry>
-                    <box size="0.9 0.08 0.3"/>
+                    <box size="1.070000 0.080000 0.300000"/>
                 </geometry>
             </collision>
             <!-- back -->
             <collision>
-                <origin xyz="-0.325 0 -0.18" rpy="0 0 0"/>
+                <origin xyz="-0.325000 0.000000 -0.180000" rpy="0 0 0"/>
                 <geometry>
-                    <box size="0.25 0.6 0.1"/>
+                    <box size="0.400000 0.645000 0.100000"/>
                 </geometry>
             </collision>
@@ -68,5 +68,5 @@
         </xacro:hokuyo_utm30lx_gpu>
         <joint name="track_left_joint" type="revolute">
-            <origin xyz="0 0 0" rpy="0 0 0"/>
+            <origin xyz="0.000000 0.000000 0.000000" rpy="0 0 0"/>
             <axis xyz="0 0 1"/>
             <parent link="talon"/>
@@ -76,12 +76,13 @@
         </joint>
         <link name="track_left">
+            <!-- dummy inertial values -->
             <inertial>
                 <mass value="0.003141"/>
-                <origin xyz="0 0 0" rpy="0 0 0"/>
+                <origin xyz="0.000000 0.000000 0.000000" rpy="0 0 0"/>
                 <inertia ixx="0.003141" ixy="0" ixz="0" iyy="0.003141" iyz="0" izz="0.003141"/>
             </inertial>
         </link>
         <joint name="track_right_joint" type="revolute">
-            <origin xyz="0 0 0" rpy="0 0 0"/>
+            <origin xyz="0.000000 0.000000 0.000000" rpy="0 0 0"/>
             <axis xyz="0 0 1"/>
             <parent link="talon"/>
@@ -91,7 +92,8 @@
         </joint>
         <link name="track_right">
+            <!-- dummy inertial values -->
             <inertial>
                 <mass value="0.003141"/>
-                <origin xyz="0 0 0" rpy="0 0 0"/>
+                <origin xyz="0.000000 0.000000 0.000000" rpy="0 0 0"/>
                 <inertia ixx="0.003141" ixy="0" ixz="0" iyy="0.003141" iyz="0" izz="0.003141"/>
             </inertial>

Commit message: move hokuyo on roman up a few centimeters
Former-commit-id: 8a72800efbcaf0ea2d1567b168962b1406256b9c

File: src/roman_model/urdf/talon.urdf.xacro (robot description, xacro)
@@ -65,5 +65,5 @@
         </link>
         <xacro:hokuyo_utm30lx_gpu name="base_laser" parent="base_link" ros_topic="base_scan" update_rate="20.0" ray_count="1080" min_angle="-130" max_angle="130">
-            <origin xyz="0.413 0 0.210" rpy="0 0 0"/>
+            <origin xyz="0.50 0 0.210" rpy="0 0 0"/>
         </xacro:hokuyo_utm30lx_gpu>
         <joint name="track_left_joint" type="revolute">

Commit message: bringin up the rear

File: src/roman_model/urdf/talon.urdf.xacro (robot description, xacro)
@@ -58,7 +58,7 @@
             <!-- back -->
             <collision>
-                <origin xyz="-0.325000 0.000000 -0.180000" rpy="0 0 0"/>
+                <origin xyz="-0.325000 0.000000 -0.280000" rpy="0 0 0"/>
                 <geometry>
-                    <box size="0.400000 0.645000 0.100000"/>
+                    <box size="0.400000 0.645000 0.300000"/>
                 </geometry>
             </collision>
