Commit message: add roman torso mesh to torso urdf
Former-commit-id: 92b4daace1ca2505a3befc2639bf1664906c9b84

File: src/roman_model/urdf/roman_body.urdf.xacro (robot description, xacro)
@@ -18,6 +18,6 @@
                 <origin xyz="0.593 0 0" rpy="1.57080 1.57080 0"/>
                 <geometry>
-                    <box size="0.1 0.1 0.1"/>
-<!--                    <mesh filename="package://roman_model/meshes/roman_torso_scaled.stl" scale="1 1 1"/> -->
+                    <!-- <box size="0.1 0.1 0.1"/> -->
+                   <mesh filename="package://roman_model/meshes/roman_torso.stl" scale="1 1 1"/>
                 </geometry>
                 <material name="grey">

Commit message: add an asus camera to the roman chest
Former-commit-id: 5fc140289b7d7ae681bd6a3c02a44d5bfc1f9143

File: src/roman_model/urdf/roman_body.urdf.xacro (robot description, xacro)
@@ -3,4 +3,5 @@
     <xacro:include filename="$(find roman_model)/gazebo/roman_body.gazebo.xacro"/>
     <xacro:include filename="$(find roman_model)/control/roman_body.transmission.xacro"/>
+    <xacro:include filename="$(find hector_sensors_description)/urdf/asus_camera.urdf.xacro"/>
     <xacro:macro name="roman_body" params="name parent *origin namespace">
         <joint name="torso_joint0" type="fixed">
@@ -63,4 +64,7 @@
             </collision>
         </link>
+        <xacro:asus_camera name="camera" parent="chest">
+            <origin xyz="0.05 -0.075 0" rpy="${-M_PI/2} 0.0 -2.09"/>
+        </xacro:asus_camera>
         <xacro:roman_body_gazebo name="${name}" namespace="${namespace}"/>
         <xacro:roman_body_transmission name="${name}" namespace="${namespace}"/>

Commit message: move silly torso cylinder to keep it from spinning robot
Former-commit-id: 7bee19294c77d6c1ae8f2ccb791b1f7ee43bc620

File: src/roman_model/urdf/roman_body.urdf.xacro (robot description, xacro)
@@ -27,5 +27,5 @@
             </visual>
             <collision>
-                <origin rpy="3.1415 -1.57080 0" xyz="-.025 0 0"/>
+                <origin rpy="3.1415 -1.57080 0" xyz="0.25 0 0"/>
                 <geometry>
                     <cylinder length="0.145" radius="0.05"/>

Commit message: integrate sensor collision volumes from sisirs urdf
Former-commit-id: f2daf59cd21de467d479bf12237396cbf311e5ca

File: src/roman_model/urdf/roman_body.urdf.xacro (robot description, xacro)
@@ -11,4 +11,5 @@
         </joint>
         <link name="torso_link0">
+            <!-- dummy inertial values -->
             <inertial>
                 <mass value="0.003141"/>
@@ -19,5 +20,4 @@
                 <origin xyz="0.593 0 0" rpy="1.57080 1.57080 0"/>
                 <geometry>
-                    <!-- <box size="0.1 0.1 0.1"/> -->
                    <mesh filename="package://roman_model/meshes/roman_torso.stl" scale="1 1 1"/>
                 </geometry>
@@ -27,12 +27,17 @@
             </visual>
             <collision>
-                <origin rpy="3.1415 -1.57080 0" xyz="0.25 0 0"/>
+                <origin xyz="0.2965 0 0" rpy="3.1415 -1.57080 0"/>
                 <geometry>
-                    <cylinder length="0.145" radius="0.05"/>
+                    <box size="0.20 0.20 0.593"/>
+                </geometry>
+            </collision>
+            <collision>
+                <origin xyz="0.2965 0.15 0" rpy="3.1415 -1.57080 0"/>
+                <geometry>
+                    <box size="0.20 0.10 0.10"/>
                 </geometry>
             </collision>
         </link>
         <joint name="torso_joint1" type="revolute">
-<!--            <origin xyz="0.17203 0 0"  rpy="3.14159 0 0"/> -->
             <origin xyz="0.593 0 0" rpy="3.14159 0 0"/>
             <axis xyz="1 0 0"/>
@@ -46,4 +51,5 @@
                 <mass value="10.0"/>
                 <origin xyz="0 0 0" rpy="0 0 0"/>
+                <!-- dummy moments -->
                 <inertia ixx="0.003141" ixy="0" ixz="0" iyy="0.003141" iyz="0" izz="0.003141"/>
             </inertial>
@@ -60,5 +66,6 @@
                 <origin xyz="0.0065 0 0" rpy="0 0 0"/>
                 <geometry>
-                    <box size="0.013 0.1 0.25"/>
+<!--                    <box size="0.013 0.1 0.25"/> -->
+                    <box size="0.013 0.4 0.4"/>
                 </geometry>
             </collision>

Commit message: add collision boxes for asus and control box

File: src/roman_model/urdf/roman_body.urdf.xacro (robot description, xacro)
@@ -70,4 +70,18 @@
                 </geometry>
             </collision>
+            <!-- asus and stuff -->
+            <collision>
+                <origin xyz="0.05 -0.1645 0.03825" rpy="0 0 0"/>
+                <geometry>
+                    <box size="0.14 0.10609 0.14"/>
+                </geometry>
+            </collision>
+            <!-- hat -->
+            <collision>
+                <origin xyz="0.20 0.03 0.0"/>
+                <geometry>
+                    <box size="0.1 0.16 0.40"/>
+                </geometry>
+            </collision>
         </link>
         <xacro:asus_camera name="asus" parent="chest">

Commit message: limit the torso rotation from -25 to 45 degs

File: src/roman_model/urdf/roman_body.urdf.xacro (robot description, xacro)
@@ -44,5 +44,8 @@
             <parent link="torso_link0"/>
             <child link="chest"/>
+<!--
             <limit effort="1000.0" lower="-6.283185" upper="6.283185" velocity="0.5"/>
+-->
+            <limit effort="1000.0" lower="-0.436" upper="0.785" velocity="0.5"/>
             <dynamics damping="1.0" friction="10.0"/>
         </joint>
