Commit message: move torso to match latest jpl urdf
Former-commit-id: 6688ced81f773dc6bf4182349d11a58e45c8ad7d

File: src/roman_model/robots/rcta_roman.urdf.xacro (robot description, xacro)
@@ -10,6 +10,7 @@
         <!--
         <origin xyz="0.27 0 -0.05" rpy="0 1.5708 1.5708"/>
+        <origin xyz="0.27 0 0.06" rpy="3.14 1.5708 1.5708"/>
         -->
-        <origin xyz="0.27 0 0.06" rpy="3.14 1.5708 1.5708"/>
+        <origin xyz="0.355000 0.000000 0.000000" rpy="3.141592 1.570800 1.570800"/>
     </xacro:roman_body>
     <!-- robosimian_l_arm origin was rpy="0 0.7854 -1.5708?"-->

Commit message: small fix to torso placement
Former-commit-id: f9ba146aa33a9a8e08b2b181d9d9381640aef4f0

File: src/roman_model/robots/rcta_roman.urdf.xacro (robot description, xacro)
@@ -12,5 +12,5 @@
         <origin xyz="0.27 0 0.06" rpy="3.14 1.5708 1.5708"/>
         -->
-        <origin xyz="0.355000 0.000000 0.000000" rpy="3.141592 1.570800 1.570800"/>
+        <origin xyz="0.355000 0.000000 0.090000" rpy="3.141592 1.570800 1.570800"/>
     </xacro:roman_body>
     <!-- robosimian_l_arm origin was rpy="0 0.7854 -1.5708?"-->
