Commit message: first pass crate object demonstration...
* only record state/move object when robot moves
* add tool frame to crate
* implement crate kinematics
* add default pose for crate in demonstrator

File: object_manipulation_planner/urdf/crate.urdf (robot description, URDF)
Before this commit: robot crate, 3 links, 2 joints
Links:
- added link tool
Joints:
- added joint tool_joint: type fixed, parent handle, child tool, origin xyz=0.0 0.0 0.0725 rpy=0 0 0
